File: summer_melt_badge_2022/summer_melt_badge_2022.kicad_sch (KiCad schematic)
At the start: 10 parts

Commit message: I made some changes to the schematic
Parts:
- added D? (x3): LED, symbol Device:LED
- R?: value 4.7k (confirm) -> 4.7k
Connections:
- net +3V0: now also S?.2; no longer BT?.1 (+)
- net GND: now also BT?.2 (-), D?.1 (K), D?.1 (K), D?.1 (K); no longer S?.1
- net GPIO0: now also D?.2 (A)
- net GPIO1: now also D?.2 (A)
- net at U?.3 (D0): now also D?.2 (A)
- new net +BATT: BT?.1 (+), S?.1
Other:
- moved on the sheet: BT?, D?, R?, S?, U?

Commit message: footprint assignment, placement started
Parts:
- removed J?: SAO, symbol Connector_Generic:Conn_02x03_Counter_Clockwise
- added J1: Conn_02x03_Odd_Even, Connector_PinSocket_2.54mm:PinSocket_2x03_P2.54mm_Vertical, symbol Connector_Generic:Conn_02x03_Odd_Even
- BT1: renamed from BT?; footprint (none) -> Battery:BatteryHolder_Keystone_2468_2xAAA
- D1, D2, D3, D4, D5, D6: renamed from D?; footprint (none) -> LED_THT:LED_D5.0mm
- H1: renamed from H?; footprint (none) -> lanyard_slot:lanyard_slot
- R1: renamed from R?; footprint (none) -> Resistor_THT:R_Axial_Power_L25.0mm_W9.0mm_P30.48mm
- S1: renamed from S?; footprint SW_SS12D07VG4 -> SS12D07VG4:SW_SS12D07VG4
- gave numbers to parts that had none: 2
Connections:
- net +3V0: now also J1.2 (Pin_2)
- net GND: now also J1.1 (Pin_1)
- net GPIO0: now also J1.6 (Pin_6)
- net GPIO1: now also J1.5 (Pin_5)
- net SCL: now also J1.3 (Pin_3)
- net SDA: now also J1.4 (Pin_4)
Other:
- note added: "LANYARD SLOT"

Commit message: draft placement complete.
Parts:
- R1: footprint Resistor_THT:R_Axial_Power_L25.0mm_W9.0mm_P30.48mm -> Resistor_THT:R_Axial_DIN0207_L6.3mm_D2.5mm_P10.16mm_Horizontal
Changed lines of the file:
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@@
     (property "Reference" "R1" (id 0) (at 116.84 78.74 90))
     (property "Value" "4.7k" (id 1) (at 116.84 81.28 90))
-    (property "Footprint" "Resistor_THT:R_Axial_Power_L25.0mm_W9.0mm_P30.48mm" (id 2) (at 116.84 85.09 0)
+    (property "Footprint" "Resistor_THT:R_Axial_DIN0207_L6.3mm_D2.5mm_P10.16mm_Horizontal" (id 2) (at 116.84 85.09 0)
       (effects (font (size 1.27 1.27)) hide)
     )
@@
     )
     (path "/dcce9beb-a6a5-4ab2-8739-7a753559b830"
-      (reference "R1") (unit 1) (value "4.7k") (footprint "Resistor_THT:R_Axial_Power_L25.0mm_W9.0mm_P30.48mm")
+      (reference "R1") (unit 1) (value "4.7k") (footprint "Resistor_THT:R_Axial_DIN0207_L6.3mm_D2.5mm_P10.16mm_Horizontal")
     )
     (path "/e8832788-83ec-4c5a-a4dd-e62560321ac4"

Commit message: final draft placement
Parts:
- removed D3: LED, LED_THT:LED_D5.0mm, symbol Device:LED
Changed lines of the file:
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@@
   (junction (at 109.22 93.98) (diameter 0) (color 0 0 0 0)
-  )
-  (junction (at 93.98 71.12) (diameter 0) (color 0 0 0 0)
   )
   (junction (at 93.98 60.96) (diameter 0) (color 0 0 0 0)
@@
     (stroke (width 0) (type default) (color 0 0 0 0))
   )
-  (wire (pts (xy 93.98 60.96) (xy 93.98 71.12))
-    (stroke (width 0) (type default) (color 0 0 0 0))
-  )
   (wire (pts (xy 83.82 93.98) (xy 76.2 93.98))
     (stroke (width 0) (type default) (color 0 0 0 0))
@@
     (stroke (width 0) (type default) (color 0 0 0 0))
   )
-  (wire (pts (xy 81.28 71.12) (xy 83.82 71.12))
-    (stroke (width 0) (type default) (color 0 0 0 0))
-  )
-  (wire (pts (xy 93.98 71.12) (xy 93.98 72.39))
-    (stroke (width 0) (type default) (color 0 0 0 0))
-  )
-  (wire (pts (xy 91.44 71.12) (xy 93.98 71.12))
+  (wire (pts (xy 93.98 60.96) (xy 93.98 72.39))
     (stroke (width 0) (type default) (color 0 0 0 0))
   )
@@
     (property "Intersheet References" "${INTERSHEET_REFS}" (id 0) (at 148.5106 74.0288 90)
       (effects (font (size 1.27 1.27)) (justify left) hide)
-    )
-  )
-  (global_label "GPIO1" (shape input) (at 81.28 71.12 180) (fields_autoplaced)
-    (effects (font (size 1.27 1.27)) (justify right))
-    (property "Intersheet References" "${INTERSHEET_REFS}" (id 0) (at 73.1821 71.0406 0)
-      (effects (font (size 1.27 1.27)) (justify right) hide)
     )
   )
@@
     (pin "2")
   )
-  (symbol (lib_id "Device:LED") (at 87.63 71.12 180) (unit 1)
-    (in_bom yes) (on_board yes) (fields_autoplaced)
-    (property "Reference" "D3" (id 0) (at 89.2175 64.9945 0))
-    (property "Value" "LED" (id 1) (at 89.2175 67.7696 0))
-    (property "Footprint" "LED_THT:LED_D5.0mm" (id 2) (at 87.63 71.12 0)
-      (effects (font (size 1.27 1.27)) hide)
-    )
-    (property "Datasheet" "~" (id 3) (at 87.63 71.12 0)
-      (effects (font (size 1.27 1.27)) hide)
-    )
-    (pin "1")
-    (pin "2")
-  )
   (symbol (lib_id "Device:R_Small_US") (at 116.84 85.09 90) (unit 1)
     (in_bom yes) (on_board yes) (fields_autoplaced)
@@
       (reference "D2") (unit 1) (value "LED") (footprint "LED_THT:LED_D5.0mm")
     )
-    (path "/ca52fe85-4ff5-40aa-bdb0-f03f3356ef70"
-      (reference "D3") (unit 1) (value "LED") (footprint "LED_THT:LED_D5.0mm")
-    )
     (path "/c7d261b6-2a48-49ba-9c79-c0f5dcd4317c"

Commit message: Minor edits during final placement review
Parts:
- renumbered D4 to D3, D5 to D4, D6 to D5
Other:
- moved on the sheet: D1, D2

Commit message: routed board review complete
Connections:
- net +3V0: now also J1.1 (Pin_1); no longer J1.2 (Pin_2)
- net GND: now also J1.2 (Pin_2); no longer J1.1 (Pin_1)
- net GPIO0: now also J1.5 (Pin_5); no longer J1.6 (Pin_6)
- net GPIO1: now also J1.6 (Pin_6); no longer J1.5 (Pin_5)
- net SCL: now also J1.4 (Pin_4); no longer J1.3 (Pin_3)
- net SDA: now also J1.3 (Pin_3); no longer J1.4 (Pin_4)
Changed lines of the file:
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@@
     )
   )
-  (global_label "GPIO1" (shape input) (at 151.13 92.71 270) (fields_autoplaced)
-    (effects (font (size 1.27 1.27)) (justify right))
-    (property "Intersheet References" "${INTERSHEET_REFS}" (id 0) (at 151.2094 100.8079 90)
+  (global_label "GPIO1" (shape input) (at 151.13 80.01 90) (fields_autoplaced)
+    (effects (font (size 1.27 1.27)) (justify left))
+    (property "Intersheet References" "${INTERSHEET_REFS}" (id 0) (at 151.2094 71.9121 90)
       (effects (font (size 1.27 1.27)) (justify right) hide)
     )
@@
     )
   )
-  (global_label "SCL" (shape input) (at 148.59 92.71 270) (fields_autoplaced)
+  (global_label "SCL" (shape input) (at 148.59 80.01 90) (fields_autoplaced)
+    (effects (font (size 1.27 1.27)) (justify left))
+    (property "Intersheet References" "${INTERSHEET_REFS}" (id 0) (at 148.6694 74.0893 90)
+      (effects (font (size 1.27 1.27)) (justify right) hide)
+    )
+  )
+  (global_label "SDA" (shape input) (at 64.77 78.74 0) (fields_autoplaced)
+    (effects (font (size 1.27 1.27)) (justify left))
+    (property "Intersheet References" "${INTERSHEET_REFS}" (id 0) (at 70.7512 78.6606 0)
+      (effects (font (size 1.27 1.27)) (justify left) hide)
+    )
+  )
+  (global_label "DQ" (shape input) (at 64.77 81.28 0) (fields_autoplaced)
+    (effects (font (size 1.27 1.27)) (justify left))
+    (property "Intersheet References" "${INTERSHEET_REFS}" (id 0) (at 69.7836 81.2006 0)
+      (effects (font (size 1.27 1.27)) (justify left) hide)
+    )
+  )
+  (global_label "GPIO0" (shape input) (at 151.13 92.71 270) (fields_autoplaced)
     (effects (font (size 1.27 1.27)) (justify right))
-    (property "Intersheet References" "${INTERSHEET_REFS}" (id 0) (at 148.6694 98.6307 90)
-      (effects (font (size 1.27 1.27)) (justify right) hide)
-    )
-  )
-  (global_label "SDA" (shape input) (at 64.77 78.74 0) (fields_autoplaced)
-    (effects (font (size 1.27 1.27)) (justify left))
-    (property "Intersheet References" "${INTERSHEET_REFS}" (id 0) (at 70.7512 78.6606 0)
-      (effects (font (size 1.27 1.27)) (justify left) hide)
-    )
-  )
-  (global_label "DQ" (shape input) (at 64.77 81.28 0) (fields_autoplaced)
-    (effects (font (size 1.27 1.27)) (justify left))
-    (property "Intersheet References" "${INTERSHEET_REFS}" (id 0) (at 69.7836 81.2006 0)
-      (effects (font (size 1.27 1.27)) (justify left) hide)
-    )
-  )
-  (global_label "GPIO0" (shape input) (at 151.13 80.01 90) (fields_autoplaced)
-    (effects (font (size 1.27 1.27)) (justify left))
-    (property "Intersheet References" "${INTERSHEET_REFS}" (id 0) (at 151.0506 71.9121 90)
+    (property "Intersheet References" "${INTERSHEET_REFS}" (id 0) (at 151.0506 100.8079 90)
       (effects (font (size 1.27 1.27)) (justify left) hide)
     )
@@
     )
   )
-  (global_label "SDA" (shape input) (at 148.59 80.01 90) (fields_autoplaced)
-    (effects (font (size 1.27 1.27)) (justify left))
-    (property "Intersheet References" "${INTERSHEET_REFS}" (id 0) (at 148.5106 74.0288 90)
+  (global_label "SDA" (shape input) (at 148.59 92.71 270) (fields_autoplaced)
+    (effects (font (size 1.27 1.27)) (justify right))
+    (property "Intersheet References" "${INTERSHEET_REFS}" (id 0) (at 148.5106 98.6912 90)
       (effects (font (size 1.27 1.27)) (justify left) hide)
     )
@@
     )
   )
-  (symbol (lib_id "power:GND") (at 146.05 92.71 0) (unit 1)
-    (in_bom yes) (on_board yes)
-    (property "Reference" "#PWR015" (id 0) (at 146.05 99.06 0)
-      (effects (font (size 1.27 1.27)) hide)
-    )
-    (property "Value" "GND" (id 1) (at 145.034 96.52 0))
-    (property "Footprint" "" (id 2) (at 146.05 92.71 0)
-      (effects (font (size 1.27 1.27)) hide)
-    )
-    (property "Datasheet" "" (id 3) (at 146.05 92.71 0)
+  (symbol (lib_id "power:GND") (at 146.05 80.01 0) (mirror x) (unit 1)
+    (in_bom yes) (on_board yes)
+    (property "Reference" "#PWR015" (id 0) (at 146.05 73.66 0)
+      (effects (font (size 1.27 1.27)) hide)
+    )
+    (property "Value" "GND" (id 1) (at 145.034 76.2 0))
+    (property "Footprint" "" (id 2) (at 146.05 80.01 0)
+      (effects (font (size 1.27 1.27)) hide)
+    )
+    (property "Datasheet" "" (id 3) (at 146.05 80.01 0)
       (effects (font (size 1.27 1.27)) hide)
     )
@@
     (pin "2")
   )
-  (symbol (lib_id "power:+3V0") (at 146.05 80.01 0) (unit 1)
-    (in_bom yes) (on_board yes)
-    (property "Reference" "#PWR014" (id 0) (at 146.05 83.82 0)
-      (effects (font (size 1.27 1.27)) hide)
-    )
-    (property "Value" "+3V0" (id 1) (at 144.272 76.2 0))
-    (property "Footprint" "" (id 2) (at 146.05 80.01 0)
-      (effects (font (size 1.27 1.27)) hide)
-    )
-    (property "Datasheet" "" (id 3) (at 146.05 80.01 0)
-      (effects (font (size 1.27 1.27)) hide)
-    )
+  (symbol (lib_id "power:+3V0") (at 146.05 92.71 0) (mirror x) (unit 1)
+    (in_bom yes) (on_board yes)
+    (property "Reference" "#PWR014" (id 0) (at 146.05 88.9 0)
+      (effects (font (size 1.27 1.27)) hide)
+    )
+    (property "Value" "+3V0" (id 1) (at 144.272 96.52 0))
+    (property "Footprint" "" (id 2) (at 146.05 92.71 0)
+      (effects (font (size 1.27 1.27)) hide)
+    )
+    (property "Datasheet" "" (id 3) (at 146.05 92.71 0)
+      (effects (font (size 1.27 1.27)) hide)
+    )
